File: psu.kicad_sch (KiCad schematic)
At the start: 7 parts

Commit message: Start layout
Parts:
- C1: renamed from CP?; LCSC C134236 -> (none)
- C2: renamed from CP?; LCSC C185774 -> (none)
- C3: renamed from CP?; LCSC C171664 -> (none)
- Q2: renamed from Q?; LCSC C53071 -> (none); Mouser (none) -> https://eu.mouser.com/ProductDetail/Diotec-Semiconductor/MM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
- R2: renamed from R?; JLC C4190 -> (none); LCSC C4190 -> (none)
- U1: renamed from U?; LCSC C579621 -> (none)
- gave numbers to parts that had none: 1
Changed lines of the file:
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@@
   (symbol (lib_id "Device:R") (at 71.12 36.83 270) (unit 1)
     (in_bom yes) (on_board yes)
-    (property "Reference" "R?" (id 0) (at 71.12 31.5722 90))
+    (property "Reference" "R2" (id 0) (at 71.12 31.5722 90))
     (property "Value" "2.2K" (id 1) (at 71.12 33.8836 90))
     (property "Footprint" "Resistor_SMD:R_0603_1608Metric_Pad0.98x0.95mm_HandSolder" (id 2) (at 71.12 35.052 90)
@@
       (effects (font (size 1.27 1.27)) hide)
     )
-    (property "JLC" "C4190" (id 4) (at 71.12 36.83 0)
+    (property "JLC" "" (id 4) (at 71.12 36.83 0)
       (effects (font (size 1.27 1.27)) hide)
     )
-    (property "LCSC" "C4190" (id 5) (at 71.12 36.83 0)
+    (property "LCSC" "" (id 5) (at 71.12 36.83 0)
       (effects (font (size 1.27 1.27)) hide)
     )
@@
   (symbol (lib_id "Device:C_Polarized") (at 74.93 62.23 0) (unit 1)
     (in_bom yes) (on_board yes)
-    (property "Reference" "CP?" (id 0) (at 77.9272 61.0616 0)
+    (property "Reference" "C2" (id 0) (at 77.9272 61.0616 0)
       (effects (font (size 1.27 1.27)) (justify left))
     )
@@
       (effects (font (size 1.27 1.27)) hide)
     )
-    (property "LCSC" "C185774" (id 4) (at 74.93 62.23 0)
+    (property "LCSC" "" (id 4) (at 74.93 62.23 0)
       (effects (font (size 1.27 1.27)) hide)
     )
@@
   (symbol (lib_id "Transistor_BJT:MMBT3904") (at 83.82 36.83 0) (unit 1)
     (in_bom yes) (on_board yes)
-    (property "Reference" "Q?" (id 0) (at 88.6714 35.6616 0)
+    (property "Reference" "Q2" (id 0) (at 88.6714 35.6616 0)
       (effects (font (size 1.27 1.27)) (justify left))
     )
@@
       (effects (font (size 1.27 1.27)) (justify left) hide)
     )
-    (property "LCSC" "C53071" (id 4) (at 83.82 36.83 0)
+    (property "LCSC" "" (id 4) (at 83.82 36.83 0)
+      (effects (font (size 1.27 1.27)) hide)
+    )
+    (property "Mouser" "https://eu.mouser.com/ProductDetail/Diotec-Semiconductor/MMFTP3401?qs=OlC7AqGiEDm4awuFJShdIQ%3D%3D" (id 5) (at 83.82 36.83 0)
       (effects (font (size 1.27 1.27)) hide)
     )
@@
   (symbol (lib_id "Device:C_Polarized") (at 45.72 55.88 0) (unit 1)
     (in_bom yes) (on_board yes)
-    (property "Reference" "CP?" (id 0) (at 48.7172 54.7116 0)
+    (property "Reference" "C1" (id 0) (at 48.7172 54.7116 0)
       (effects (font (size 1.27 1.27)) (justify left))
     )
@@
       (effects (font (size 1.27 1.27)) hide)
     )
-    (property "LCSC" "C134236" (id 4) (at 45.72 55.88 0)
+    (property "LCSC" "" (id 4) (at 45.72 55.88 0)
       (effects (font (size 1.27 1.27)) hide)
     )
@@
   (symbol (lib_id "Device:C_Polarized") (at 86.36 55.88 180) (unit 1)
     (in_bom yes) (on_board yes)
-    (property "Reference" "CP?" (id 0) (at 89.3572 54.7116 0)
+    (property "Reference" "C3" (id 0) (at 89.3572 54.7116 0)
       (effects (font (size 1.27 1.27)) (justify right))
     )
@@
       (effects (font (size 1.27 1.27)) hide)
     )
-    (property "LCSC" "C171664" (id 4) (at 86.36 55.88 0)
+    (property "LCSC" "" (id 4) (at 86.36 55.88 0)
       (effects (font (size 1.27 1.27)) hide)
     )
@@
   (symbol (lib_id "Regulator_SwitchedCapacitor:LT1054") (at 63.5 59.69 0) (unit 1)
     (in_bom yes) (on_board yes)
-    (property "Reference" "U?" (id 0) (at 63.5 45.2882 0))
+    (property "Reference" "U1" (id 0) (at 63.5 45.2882 0))
     (property "Value" "LT1054" (id 1) (at 63.5 47.5996 0))
     (property "Footprint" "Package_SO:SOIC-8_3.9x4.9mm_P1.27mm" (id 2) (at 66.04 62.23 0)
@@
       (effects (font (size 1.27 1.27)) hide)
     )
-    (property "LCSC" "C579621" (id 4) (at 63.5 59.69 0)
+    (property "LCSC" "" (id 4) (at 63.5 59.69 0)
       (effects (font (size 1.27 1.27)) hide)
     )
@@
   (symbol (lib_id "Connector:TestPoint") (at 97.79 25.4 0) (unit 1)
     (in_bom yes) (on_board yes)
-    (property "Reference" "TP?" (id 0) (at 99.2632 22.4028 0)
+    (property "Reference" "TP1" (id 0) (at 99.2632 22.4028 0)
       (effects (font (size 1.27 1.27)) (justify left))
     )
