File: line-driver.kicad_sch (KiCad schematic)
At the start: 0 parts

Commit message: Start layout
Parts:
- added C13, C14: 10u, Capacitor_SMD:C_1206_3216Metric_Pad1.33x1.80mm_HandSolder, symbol Device:C
- added C15, C16, C17, C18, C19, C20: 100n, Capacitor_SMD:C_0603_1608Metric_Pad1.08x0.95mm_HandSolder, symbol Device:C
- added D10, D11, D8, D9: FM4004-W, Diode_SMD:D_SMA, symbol Diode:MRA4004T3G
- added FB1, FB2: FerriteBead, Resistor_SMD:R_0603_1608Metric_Pad0.98x0.95mm_HandSolder, symbol Device:FerriteBead
- added R12: 1k, Resistor_SMD:R_0603_1608Metric_Pad0.98x0.95mm_HandSolder, symbol Device:R
- added R13: 10, Resistor_SMD:R_0603_1608Metric_Pad0.98x0.95mm_HandSolder, symbol Device:R
- added RV2: A20K, R0904NB10KL-25KQ:V3_TRIM_R0904NB10KL-Keepout, symbol R0904NB10KL-25KQ:R_Potentiometer_Shield
- added TP5: Vol_Out, TestPoint:TestPoint_THTPad_D1.5mm_Drill0.7mm, symbol Connector:TestPoint
- added TP6: 1646_Out+, TestPoint:TestPoint_THTPad_D1.5mm_Drill0.7mm, symbol Connector:TestPoint
- added TP7: 1646_Out-, TestPoint:TestPoint_THTPad_D1.5mm_Drill0.7mm, symbol Connector:TestPoint
- added U3: NE5532, Package_SO:SOIC-8_3.9x4.9mm_P1.27mm, symbol Amplifier_Operational:NE5532
- added U4: THAT1646, Package_SO:SOIC-8_3.9x4.9mm_P1.27mm, symbol pedals:THAT1646
Connections:
- new net: RV2.2, TP5.1, U3.3 (+), U3.5 (+)
- new net: C14.1, U4.2 (Sns-)
- new net: C13.1, U4.7 (Sns+)
- new net: R13.2, U4.4 (In)
- new net: R13.1, U3.6 (-), U3.7
- new net: R12.1, U3.1, U3.2 (-)
- new net GND: C15.1, C16.2, C17.1, C18.1, C19.1, C20.1, RV2.0 (ShieldPin), RV2.1, U4.3 (GND)
- new net In: RV2.3
- new net InstrumentOut: R12.2
- new net LineOut+: C13.2, D10.1 (K), D8.2 (A), FB1.1, TP6.1, U4.8 (Out+)
- new net LineOut-: C14.2, D11.1 (K), D9.2 (A), FB2.1, TP7.1, U4.1 (Out-)
- new net Out+: C15.2, FB1.2
- new net Out-: C16.1, FB2.2
- new net V+: C17.2, C18.2, D8.1 (K), D9.1 (K), U3.8 (V+), U4.6 (V+)
- new net V-: C19.2, C20.2, D10.2 (A), D11.2 (A), U3.4 (V-), U4.5 (V-)

Commit message: Layout draft done
Parts:
- D10, D11, D8, D9: footprint Diode_SMD:D_SMA -> Diode_SMD:D_SMA_Handsoldering
Changed lines of the file:
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@@
       (effects (font (size 1.27 1.27)) (justify left))
     )
-    (property "Footprint" "Diode_SMD:D_SMA" (id 2) (at 122.555 73.66 0)
+    (property "Footprint" "Diode_SMD:D_SMA_Handsoldering" (id 2) (at 122.555 73.66 0)
       (effects (font (size 1.27 1.27)) hide)
     )
@@
       (effects (font (size 1.27 1.27)) (justify right))
     )
-    (property "Footprint" "Diode_SMD:D_SMA" (id 2) (at 131.445 62.23 0)
+    (property "Footprint" "Diode_SMD:D_SMA_Handsoldering" (id 2) (at 131.445 62.23 0)
       (effects (font (size 1.27 1.27)) hide)
     )
@@
       (effects (font (size 1.27 1.27)) (justify left))
     )
-    (property "Footprint" "Diode_SMD:D_SMA" (id 2) (at 147.955 62.23 0)
+    (property "Footprint" "Diode_SMD:D_SMA_Handsoldering" (id 2) (at 147.955 62.23 0)
       (effects (font (size 1.27 1.27)) hide)
     )
@@
       (effects (font (size 1.27 1.27)) (justify right))
     )
-    (property "Footprint" "Diode_SMD:D_SMA" (id 2) (at 156.845 73.66 0)
+    (property "Footprint" "Diode_SMD:D_SMA_Handsoldering" (id 2) (at 156.845 73.66 0)
       (effects (font (size 1.27 1.27)) hide)
     )
