File: pre.kicad_sch (KiCad schematic)
At the start: 25 parts

Commit message: Start layout
Parts:
- removed C? (x2): 3.3u, symbol Device:C_Polarized
- added C10, C9: 3.3u, Capacitor_SMD:C_1206_3216Metric_Pad1.33x1.80mm_HandSolder, symbol Device:C
- added C11, C12: 100n, Capacitor_SMD:C_0603_1608Metric_Pad1.08x0.95mm_HandSolder, symbol Device:C
- added TP3: 1510_In+, TestPoint:TestPoint_THTPad_D1.5mm_Drill0.7mm, symbol Connector:TestPoint
- added TP4: 1510_In-, TestPoint:TestPoint_THTPad_D1.5mm_Drill0.7mm, symbol Connector:TestPoint
- C4, C5, C6: renamed from C?; footprint (none) -> Capacitor_SMD:C_0603_1608Metric_Pad1.08x0.95mm_HandSolder
- C7, C8: renamed from C?; footprint (none) -> Capacitor_SMD:CP_Elec_4x5.4
- D6, D7: renamed from D?; footprint (none) -> Diode_SMD:D_SOD-323_HandSoldering; Mouser (none) -> https://eu.mouser.com/ProductDetail/Micro-Commercial-Compon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
- R10, R11, R3, R4, R5, R6, R7, R8, R9: renamed from R?; footprint (none) -> Resistor_SMD:R_0603_1608Metric_Pad0.98x0.95mm_HandSolder
- RV1: renamed from RV?; footprint (none) -> R0904NB10KL-25KQ:V3_TRIM_R0904NB10KL-Keepout; symbol Device:R_Potentiometer_MountingPin -> R0904NB10KL-25KQ:R_Potentiometer_Shield
- gave numbers to parts that had none: 6
Connections:
- net GND: now also RV1.0 (ShieldPin), C11.1, C12.1; no longer RV1.MP (MountPin)
- net Out: now also C10.2
- net Rg2: now also C9.2
- net V+: now also C11.2
- net V-: now also C12.2
- net InAC-: now reaches C8.2, R6.1
- net InPre-: now reaches D3.2 (A), D5.1 (K), D7.1 (K), R6.2, R8.2, U2.3 (IN2)
- net InPre-: now also TP4.1
- net InPre+: now reaches D2.2 (A), D4.1 (K), D6.1 (K), R5.2, R7.1, U2.2 (IN1)
- net InPre+: now also TP3.1
- net at R10.1: now also C9.1
- net InAC+: now reaches C7.2, R5.1
- net at TP2.1, U2.6 (Out): now also C10.1

Commit message: Layout draft done
Parts:
- C7, C8: footprint Capacitor_SMD:CP_Elec_4x5.4 -> Capacitor_SMD:CP_Elec_6.3x5.8
- D2, D3, D4, D5: footprint Diode_SMD:D_SMA -> Diode_SMD:D_SMA_Handsoldering
Changed lines of the file:
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@@
     (property "Reference" "C8" (id 0) (at 81.661 63.5 90))
     (property "Value" "22u" (id 1) (at 81.661 66.04 90))
-    (property "Footprint" "Capacitor_SMD:CP_Elec_4x5.4" (id 2) (at 86.36 70.1548 0)
+    (property "Footprint" "Capacitor_SMD:CP_Elec_6.3x5.8" (id 2) (at 86.36 70.1548 0)
       (effects (font (size 1.27 1.27)) hide)
     )
@@
       (effects (font (size 1.27 1.27)) (justify right))
     )
-    (property "Footprint" "Diode_SMD:D_SMA" (id 2) (at 142.875 66.04 0)
+    (property "Footprint" "Diode_SMD:D_SMA_Handsoldering" (id 2) (at 142.875 66.04 0)
       (effects (font (size 1.27 1.27)) hide)
     )
@@
       (effects (font (size 1.27 1.27)) (justify right))
     )
-    (property "Footprint" "Diode_SMD:D_SMA" (id 2) (at 116.205 55.88 0)
+    (property "Footprint" "Diode_SMD:D_SMA_Handsoldering" (id 2) (at 116.205 55.88 0)
       (effects (font (size 1.27 1.27)) hide)
     )
@@
       (effects (font (size 1.27 1.27)) (justify left))
     )
-    (property "Footprint" "Diode_SMD:D_SMA" (id 2) (at 107.315 66.04 0)
+    (property "Footprint" "Diode_SMD:D_SMA_Handsoldering" (id 2) (at 107.315 66.04 0)
       (effects (font (size 1.27 1.27)) hide)
     )
@@
       (effects (font (size 1.27 1.27)) (justify left))
     )
-    (property "Footprint" "Diode_SMD:D_SMA" (id 2) (at 133.985 55.88 0)
+    (property "Footprint" "Diode_SMD:D_SMA_Handsoldering" (id 2) (at 133.985 55.88 0)
       (effects (font (size 1.27 1.27)) hide)
     )
@@
     (property "Reference" "C7" (id 0) (at 81.661 43.18 90))
     (property "Value" "22u" (id 1) (at 81.661 45.72 90))
-    (property "Footprint" "Capacitor_SMD:CP_Elec_4x5.4" (id 2) (at 86.36 49.8348 0)
-      (effects (font (size 1.27 1.27)) hide)
-    )
+    (property "Footprint" "Capacitor_SMD:CP_Elec_6.3x5.8" (id 2) (at 86.36 49.8348 0)
+      (effects (font (size 1.27 1.27)) hide)
+    )
