File: preamp-test.kicad_sch (KiCad schematic)
At the start: 12 parts

Commit message: Start layout
Parts:
- D1: renamed from D?; footprint Diode_THT:D_A-405_P7.62mm_Horizontal -> Diode_SMD:D_SOD-323_HandSoldering; Mouser (none) -> https://eu.mouser.com/ProductDetail/Micro-Commercial-Compon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
- J6: renamed from J?; value Snd -> Out
- J7: renamed from J?; footprint (none) -> Connector_PinSocket_2.54mm:PinSocket_1x02_P2.54mm_Vertical
- Q1: renamed from Q?; value Q_PMOS_SGD -> MMFTP3401; footprint Package_TO_SOT_THT:TO-92L_Inline_Wide -> Package_TO_SOT_SMD:SOT-23; symbol Device:Q_PMOS_SGD -> Device:Q_PMOS_GSD
- SW1: renamed from SW?; footprint (none) -> switches:SPDT.LUGS
- SW2: renamed from SW?; footprint (none) -> switches:DPDT.LUGS
- gave numbers to parts that had none: 6
Connections:
- net +9V: now also Q1.2 (S); no longer Q1.1 (S)
- net GND: now also J7.1 (Pin_1); no longer J7.2 (Pin_2)
- net Phantom: now also J7.2 (Pin_2); no longer J7.1 (Pin_1)
- net at D1.2 (A), R1.2: now also Q1.1 (G); no longer Q1.2 (G)
Other:
- sheet Line Driver ports: added GND, In, InstrumentOut, Out+, Out-, V+, V-; removed none

Commit message: Layout draft done
Parts:
- removed J1: +9v, Connector_JST:JST_XH_B2B-XH-A_1x02_P2.50mm_Vertical, symbol Connector:Conn_01x02_Male
- removed J2: In, Connector_Audio:Jack_XLR_Neutrik_NC3FAH-0_Horizontal, symbol Connector:XLR3
- removed J3: Ret, tayda-6mm35-jack-pcb-compact:tayda-6mm35-jack-pcb-compact, symbol Connector:AudioJack3_SwitchTR
- removed J4: Out, Connector_Audio:Jack_XLR_Neutrik_NC3MAH-0_Horizontal, symbol Connector:XLR3_Ground
- removed J5: Snd, tayda-6mm35-jack-pcb-compact:tayda-6mm35-jack-pcb-compact, symbol Connector:AudioJack3_SwitchTR
- removed J6: Out, tayda-6mm35-jack-pcb-compact:tayda-6mm35-jack-pcb-compact, symbol Connector:AudioJack3_SwitchTR
- removed J7: Conn_01x02, Connector_PinSocket_2.54mm:PinSocket_1x02_P2.54mm_Vertical, symbol Connector_Generic:Conn_01x02
- added J1: Conn_01x03_Female, Connector_PinSocket_2.54mm:PinSocket_1x03_P2.54mm_Vertical, symbol Connector:Conn_01x03_Female
- added J8, J9: Conn_01x08_Male, Connector_Molex:Molex_Picoflex_90814-0008_2x04_P1.27mm_Vertical, symbol Connector:Conn_01x08_Male
- R1: footprint Resistor_THT:R_Axial_DIN0207_L6.3mm_D2.5mm_P7.62mm_Horizontal -> Resistor_SMD:R_0603_1608Metric_Pad0.98x0.95mm_HandSolder
Connections:
- net +9V: now also J1.1 (Pin_1)
- net GND: now also J1.2 (Pin_2), J8.2 (Pin_2), J8.4 (Pin_4), J8.8 (Pin_8), J9.2 (Pin_2), J9.5 (Pin_5), J9.7 (Pin_7)
- net In+: now also J8.7 (Pin_7)
- net In-: now also J8.6 (Pin_6)
- net InGND: now also J8.5 (Pin_5)
- net InstOut: now also J9.6 (Pin_6)
- net Out+: now also J9.4 (Pin_4)
- net Out-: now also J9.3 (Pin_3)
- net Phantom: now also J1.3 (Pin_3)
- net PreOut: now also J8.3 (Pin_3)
- net VolumeIn: now also J9.8 (Pin_8)
- net +9VIn renamed Jack9V
- net Jack9V: now also J9.1 (Pin_1)
- no-connect marks 9 -> 2

Commit message: More ext options
Parts:
- removed J1: Conn_01x03_Female, Connector_PinSocket_2.54mm:PinSocket_1x03_P2.54mm_Vertical, symbol Connector:Conn_01x03_Female
- added J1: Conn_01x08_Female, Connector_PinSocket_2.54mm:PinSocket_1x08_P2.54mm_Vertical, symbol Connector:Conn_01x08_Female
Connections:
- net +9V: now also J1.3 (Pin_3)
- net -9V: now also J1.1 (Pin_1)
- net GND: now also J1.2 (Pin_2), J1.5 (Pin_5), J1.8 (Pin_8)
- net Phantom: now also J1.4 (Pin_4)
- net PreOut: now also J1.6 (Pin_6); no longer J8.3 (Pin_3)
- new net Snd: J1.7 (Pin_7), J8.3 (Pin_3)
