File: preamp-test.kicad_pcb (KiCad board)
At the start: 2 copper layers, 71 parts, among them J1 +9v, J2 In, J3 Ret, J4 Out, J5 Snd, J6 Out, J7 Conn_01x02, Q1 MMFTP3401, Q2 FMMT619, SW1 GND Lift, SW2 Phase, U1 LT1054, U2 THAT1510, U3 NE5532, U4 THAT1646

Commit message: Layout draft done
Parts:
- removed J2: In, Connector_Audio:Jack_XLR_Neutrik_NC3FAH-0_Horizontal
- removed J3: Ret, tayda-6mm35-jack-pcb-compact:tayda-6mm35-jack-pcb-compact
- removed J4: Out, Connector_Audio:Jack_XLR_Neutrik_NC3MAH-0_Horizontal
- removed J5: Snd, tayda-6mm35-jack-pcb-compact:tayda-6mm35-jack-pcb-compact
- removed J6: Out, tayda-6mm35-jack-pcb-compact:tayda-6mm35-jack-pcb-compact
- removed J7: Conn_01x02, Connector_PinSocket_2.54mm:PinSocket_1x02_P2.54mm_Vertical
- added J8: Conn_01x08_Male, Connector_Molex:Molex_Picoflex_90814-0008_2x04_P1.27mm_Vertical, B.Cu at (146.5, 93.5)
- added J9: Conn_01x08_Male, Connector_Molex:Molex_Picoflex_90814-0008_2x04_P1.27mm_Vertical, B.Cu at (53.5, 93.5)
- added kibuzzard-66CA6E97: G***, kibuzzard-66CA6E97, F.Cu at (53.3, 95.1)
- added kibuzzard-66CA6ECA: G***, kibuzzard-66CA6ECA, F.Cu at (80.3, 95.1)
- added kibuzzard-66CA6F29: G***, kibuzzard-66CA6F29, F.Cu at (121.9, 95.1)
- added kibuzzard-66CA6F40: G***, kibuzzard-66CA6F40, F.Cu at (146.7, 95.1)
- C1, C10, C11, C12, C13, C14, C15, C16, C17, C18, C19, C2, C20, C3, C4, C5, C6, C9, D1, D6, D7, FB1, FB2, Q1, Q2, R10, R11, R12, R13, R2, R3, R4, R5, R6, R7, R8, R9, TP1, TP2, TP3, TP4, TP5, TP6, TP7, U1, U2, U3, U4: moved to B.Cu
- C7, C8: footprint Capacitor_SMD:CP_Elec_4x5.4 -> Capacitor_SMD:CP_Elec_6.3x5.8; moved to B.Cu
- D10, D11, D2, D3, D4, D5, D8, D9: footprint Diode_SMD:D_SMA -> Diode_SMD:D_SMA_Handsoldering; moved to B.Cu
- J1: value +9v -> Conn_01x03_Female; footprint Connector_JST:JST_XH_B2B-XH-A_1x02_P2.50mm_Vertical -> Connector_PinSocket_2.54mm:PinSocket_1x03_P2.54mm_Vertical; moved to B.Cu
- R1: footprint Resistor_THT:R_Axial_DIN0207_L6.3mm_D2.5mm_P7.62mm_Horizontal -> Resistor_SMD:R_0603_1608Metric_Pad0.98x0.95mm_HandSolder; moved to B.Cu
- moved TP1 230.1 mm to (87.3, 117.1), turned to 180 degrees
- moved Q2 222.7 mm to (87.3, 121.7), turned to -90 degrees
- moved Q1 217.7 mm to (43.4, 81.0), turned to -90 degrees
- moved U1 213.3 mm to (99.0, 117.6), turned to 180 degrees
- moved R2 213.1 mm to (83.8, 119.1), turned to 90 degrees
- moved C3 212.3 mm to (91.6, 122.0), turned to 90 degrees
- moved C15 210.9 mm to (50.5, 107.7), turned to 90 degrees
- moved C17 207.1 mm to (50.5, 117.3), turned to 90 degrees
- moved C1 206.9 mm to (91.6, 113.9), turned to 90 degrees
- moved TP6 206.2 mm to (43.7, 105.4), turned to 180 degrees
- moved D10 205.1 mm to (41.1, 113.3), turned to -90 degrees
- moved D8 204.9 mm to (46.2, 113.3), turned to 90 degrees
- moved TP5 204.3 mm to (61.7, 84.8), turned to 180 degrees
- moved FB1 203.2 mm to (54.4, 107.7), turned to 90 degrees
- moved C19 201.1 mm to (54.4, 119.9), turned to 90 degrees
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Connections:
- J1 pad 1: /GND -> /+9V
- J1 pad 2: /+9VIn -> /GND
- Q1 pad 3: /+9VIn -> /Jack9V
Routing:
- net /PreOut: track 0.00 -> 125.0 mm, vias 0 -> 2
- net Net-(R13-Pad2): track 0.00 -> 102.9 mm
- net /Preamp/InAC-: track 0.00 -> 69.1 mm
- net /Preamp/InAC+: track 0.00 -> 68.1 mm
- net /Preamp/InPre+: track 0.00 -> 53.6 mm
- net /Preamp/Rg1: track 0.00 -> 50.3 mm
- net /GND: track 0.00 -> 46.5 mm, vias 0 -> 34
- net /Phantom: track 0.00 -> 42.6 mm, vias 0 -> 2
- net /+9V: track 0.00 -> 41.8 mm, vias 0 -> 8
- net /-9V: track 0.00 -> 39.3 mm, vias 0 -> 10
- net /Sig+: track 0.00 -> 37.4 mm
- net /Sig-: track 0.00 -> 37.0 mm
- net /Preamp/InPre-: track 0.00 -> 35.5 mm
- net /InstOut: track 0.00 -> 35.5 mm
- net /InGND: track 0.00 -> 31.3 mm, vias 0 -> 1
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- added copper zone on F.Cu, net /+9V
- added copper zone on B.Cu, net /-9V
- added copper zone on In1.Cu, net /GND
- added copper zone on In2.Cu, net /GND
Other:
- board outline added: 126 x 61 mm
- copper layers 2 -> 4
- board text added: "JLCJLCJLCJLC"

Commit message: More ext options
Parts:
- added kibuzzard-66CB7A1F: G***, kibuzzard-66CB7A1F, B.Cu at (138.2, 125.3)
- added kibuzzard-66CB7A30: G***, kibuzzard-66CB7A30, B.Cu at (148.5, 125.3)
- added kibuzzard-66CB7A30: G***, kibuzzard-66CB7A30, B.Cu at (140.8, 125.3)
- added kibuzzard-66CB7A30: G***, kibuzzard-66CB7A30, B.Cu at (156.1, 125.3)
- added kibuzzard-66CB7A55: G***, kibuzzard-66CB7A55, B.Cu at (143.4, 125.3)
- added kibuzzard-66CB7AA0: G***, kibuzzard-66CB7AA0, B.Cu at (145.9, 125.3)
- added kibuzzard-66CB7AA6: G***, kibuzzard-66CB7AA6, B.Cu at (151.0, 125.3)
- added kibuzzard-66CB7AAB: G***, kibuzzard-66CB7AAB, B.Cu at (153.5, 125.3)
- J1: value Conn_01x03_Female -> Conn_01x08_Female; footprint Connector_PinSocket_2.54mm:PinSocket_1x03_P2.54mm_Vertical -> Connector_PinSocket_2.54mm:PinSocket_1x08_P2.54mm_Vertical
- moved J1 9.23 mm to (138.3, 121.5), turned to -90 degrees
Connections:
- J1 pad 1: /+9V -> /-9V
- J1 pad 3: /Phantom -> /+9V
- J8 pad 3: /PreOut -> /Snd
Routing:
- net /Snd: track 0.00 -> 53.1 mm, vias 0 -> 2
- net /PreOut: track 125.0 -> 176.5 mm, vias 2 -> 0
- net /-9V: track 39.3 -> 24.9 mm, vias 10 -> 4
- net /Phantom: track 42.6 -> 39.8 mm
- net /GND: vias 34 -> 31

Commit message: Ordered at JLC
Parts:
- added kibuzzard-66CB7C93: G***, kibuzzard-66CB7C93, B.Cu at (100.0, 128.5)
