File: preamp-test-jacks-board/preamp-test-jacks-board.kicad_pcb (KiCad board)
At the start: 2 copper layers, 126 x 31 mm, 14 parts, among them J1 Barrel_Jack_Switch, J2 In, J3 Ret, J4 Out, J5 Snd, J6 Out, J7 Conn_01x08_Male, J8 Conn_01x08_Male

Commit message: Ordered at JLC
Parts:
- added kibuzzard-66CB7BC6: G***, kibuzzard-66CB7BC6, F.Cu at (158.0, 59.5)
- added kibuzzard-66CB7C17: G***, kibuzzard-66CB7C17, B.Cu at (109.5, 44.5)
Changed lines of the file:
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@@
+      ) (layer "F.SilkS") (width 0) (fill solid))
+  )
+  (footprint "kibuzzard-66CB7BC6" (layer "F.Cu")
+    (at 158 59.5)
+    (descr "Generated with KiBuzzard")
+    (tags "kb_params=eyJBbGlnbm1lbnRDaG9pY2UiOiAiQ2VudGVyIiwgIkNhcExlZnRDaG9pY2UiOiAiIiwgIkNhcFJpZ2h0Q2hvaWNlIjogIiIsICJGb250Q29tYm9Cb3giOiAiTW9kZXJhdC1Nb25vLU1lZGl1bSIsICJIZWlnaHRDdHJsIjogIjIiLCAiTGF5ZXJDb21ib0JveCI6ICJGLlNpbGtTIiwgIk11bHRpTGluZVRleHQiOiAiSU4iLCAiUGFkZGluZ0JvdHRvbUN0cmwiOiAiNSIsICJQYWRkaW5nTGVmdEN0cmwiOiAiNSIsICJQYWRkaW5nUmlnaHRDdHJsIjogIjUiLCAiUGFkZGluZ1RvcEN0cmwiOiAiNSIsICJXaWR0aEN0cmwiOiAiMTQuNCJ9")
+    (attr board_only exclude_from_pos_files exclude_from_bom)
+    (fp_text reference "kibuzzard-66CB7BC6" (at 0 -4.15925) (layer "F.SilkS") hide
+      (effects (font (size 0 0) (thickness 0.15)))
+    )
+    (fp_text value "G***" (at 0 4.15925) (layer "F.SilkS") hide
+      (effects (font (size 0 0) (thickness 0.15)))
+    )
+    (fp_poly (pts
+        (xy 1.368425 -1.11125)
+        (xy 1.679575 -1.11125)
+        (xy 1.679575 1.11125)
+        (xy 1.343025 1.11125)
+        (xy 0.55245 -0.47625)
+        (xy 0.530225 -0.47625)
+        (xy 0.530225 1.11125)
+        (xy 0.219075 1.11125)
+        (xy 0.219075 -1.11125)
+        (xy 0.555625 -1.11125)
+        (xy 1.3462 0.479425)
+        (xy 1.368425 0.479425)
+        (xy 1.368425 -1.11125)
+      ) (layer "F.SilkS") (width 0) (fill solid))
+    (fp_poly (pts
+        (xy -0.7874 0.815975)
+        (xy -0.23495 0.815975)
+        (xy -0.23495 1.11125)
+        (xy -1.679575 1.11125)
+        (xy -1.679575 0.815975)
+        (xy -1.120775 0.815975)
+        (xy -1.120775 -0.815975)
+        (xy -1.6637 -0.815975)
+        (xy -1.6637 -1.11125)
+        (xy -0.250825 -1.11125)
+        (xy -0.250825 -0.815975)
+        (xy -0.7874 -0.815975)
+        (xy -0.7874 0.815975)
       ) (layer "F.SilkS") (width 0) (fill solid))
   )
@@
       ) (layer "B.SilkS") (width 0) (fill solid))
   )
+  (footprint "kibuzzard-66CB7C17" (layer "B.Cu")
+    (at 109.5 44.5 180)
+    (descr "Generated with KiBuzzard")
+    (tags "kb_params=eyJBbGlnbm1lbnRDaG9pY2UiOiAiQ2VudGVyIiwgIkNhcExlZnRDaG9pY2UiOiAiIiwgIkNhcFJpZ2h0Q2hvaWNlIjogIiIsICJGb250Q29tYm9Cb3giOiAiTW9kZXJhdC1Nb25vLU1lZGl1bSIsICJIZWlnaHRDdHJsIjogIjEuMiIsICJMYXllckNvbWJvQm94IjogIkYuU2lsa1MiLCAiTXVsdGlMaW5lVGV4dCI6ICJ2MXJldjEiLCAiUGFkZGluZ0JvdHRvbUN0cmwiOiAiNSIsICJQYWRkaW5nTGVmdEN0cmwiOiAiNSIsICJQYWRkaW5nUmlnaHRDdHJsIjogIjUiLCAiUGFkZGluZ1RvcEN0cmwiOiAiNSIsICJXaWR0aEN0cmwiOiAiMTQuNCJ9")
+    (attr board_only exclude_from_pos_files exclude_from_bom)
+    (fp_text reference "kibuzzard-66CB7C17" (at 0 3.667125) (layer "B.SilkS") hide
+      (effects (font (size 0 0) (thickness 0.15)) (justify mirror))
+    )
+    (fp_text value "G***" (at 0 -3.667125) (layer "B.SilkS") hide
+      (effects (font (size 0 0) (thickness 0.15)) (justify mirror))
+    )
+    (fp_poly (pts
+        (xy 2.99466 -0.43815)
+        (xy 3.305175 -0.43815)
+        (xy 3.305175 -0.600075)
+        (xy 2.474595 -0.600075)
+        (xy 2.474595 -0.43815)
+        (xy 2.794635 -0.43815)
+        (xy 2.794635 0.24384)
+        (xy 2.50698 0.24384)
+        (xy 2.50698 0.401955)
+        (xy 2.64414 0.401955)
+        (xy 2.73939 0.4191)
+        (xy 2.79654 0.470535)
+        (xy 2.81559 0.55626)
+        (xy 2.81559 0.619125)
+        (xy 2.99466 0.619125)
+        (xy 2.99466 -0.43815)
+      ) (layer "B.SilkS") (width 0) (fill solid))
+    (fp_poly (pts
+        (xy 0.619125 -0.46101)
+        (xy 0.72898 -0.444712)
+        (xy 0.807085 -0.395817)
+        (xy 0.85344 -0.314325)
+        (xy 1.04013 -0.314325)
+        (xy 0.989171 -0.441722)
+        (xy 0.897255 -0.538163)
+        (xy 0.771525 -0.598884)
+        (xy 0.619125 -0.619125)
+        (xy 0.49022 -0.604203)
+        (xy 0.377825 -0.559435)
+        (xy 0.28194 -0.484823)
+        (xy 0.208915 -0.38608)
+        (xy 0.1651 -0.268923)
+        (xy 0.150495 -0.13335)
+        (xy 0.1651 0.008996)
+        (xy 0.208915 0.131233)
+        (xy 0.28194 0.233362)
+        (xy 0.376767 0.310092)
+        (xy 0.485987 0.356129)
+        (xy 0.6096 0.371475)
+        (xy 0.726969 0.357717)
+        (xy 0.830157 0.316442)
+        (xy 0.919162 0.24765)
+        (xy 0.987425 0.152823)
+        (xy 1.028383 0.033443)
+        (xy 1.042035 -0.11049)
+        (xy 1.038225 -0.173355)
+        (xy 0.33909 -0.173355)
+        (xy 0.33909 -0.036195)
+        (xy 0.855345 -0.036195)
+        (xy 0.837009 0.064056)
+        (xy 0.785813 0.143827)
+        (xy 0.707946 0.195977)
+        (xy 0.6096 0.21336)
+        (xy 0.511016 0.195501)
+        (xy 0.428625 0.141922)
+        (xy 0.369094 0.061674)
+        (xy 0.33909 -0.036195)
+        (xy 0.33909 -0.173355)
+        (xy 0.337185 -0.173355)
+        (xy 0.36195 -0.290274)
+        (xy 0.421005 -0.381953)
+        (xy 0.508635 -0.441246)
+        (xy 0.619125 -0.46101)
+      ) (layer "B.SilkS") (width 0) (fill solid))
+    (fp_poly (pts
+        (xy -2.54508 0.352425)
+        (xy -2.34696 0.352425)
+        (xy -2.707005 -0.600075)
+        (xy -2.943225 -0.600075)
+        (xy -3.305175 0.352425)
+        (xy -3.10515 0.352425)
+        (xy -2.83083 -0.398145)
+        (xy -2.817495 -0.398145)
+        (xy -2.54508 0.352425)
+      ) (layer "B.SilkS") (width 0) (fill solid))
+    (fp_poly (pts
+        (xy -0.177165 0.18288)
+        (xy -0.315516 0.162401)
+        (xy -0.421958 0.100965)
+        (xy -0.489823 0.00381)
+        (xy -0.512445 -0.123825)
+        (xy -0.512445 -0.45339)
+        (xy -0.1524 -0.45339)
+        (xy -0.1524 -0.600075)
+        (xy -0.984885 -0.600075)
+        (xy -0.984885 -0.45339)
+        (xy -0.706755 -0.45339)
+        (xy -0.706755 0.20574)
+        (xy -0.97536 0.20574)
+        (xy -0.97536 0.352425)
+        (xy -0.5334 0.352425)
+        (xy -0.51435 0.19431)
+        (xy -0.501015 0.19431)
+        (xy -0.442436 0.272415)
+        (xy -0.36957 0.32766)
+        (xy -0.271939 0.360521)
+        (xy -0.139065 0.371475)
+        (xy -0.066675 0.371475)
+        (xy -0.066675 0.177165)
+        (xy -0.177165 0.18288)
+      ) (layer "B.SilkS") (width 0) (fill solid))
+    (fp_poly (pts
+        (xy -1.57734 -0.43815)
+        (xy -1.266825 -0.43815)
+        (xy -1.266825 -0.600075)
+        (xy -2.097405 -0.600075)
+        (xy -2.097405 -0.43815)
+        (xy -1.777365 -0.43815)
+        (xy -1.777365 0.24384)
+        (xy -2.06502 0.24384)
+        (xy -2.06502 0.401955)
+        (xy -1.92786 0.401955)
+        (xy -1.83261 0.4191)
+        (xy -1.77546 0.470535)
+        (xy -1.75641 0.55626)
+        (xy -1.75641 0.619125)
+        (xy -1.57734 0.619125)
+        (xy -1.57734 -0.43815)
+      ) (layer "B.SilkS") (width 0) (fill solid))
+    (fp_poly (pts
+        (xy 2.02692 0.352425)
+        (xy 2.22504 0.352425)
+        (xy 1.864995 -0.600075)
+        (xy 1.628775 -0.600075)
+        (xy 1.266825 0.352425)
+        (xy 1.46685 0.352425)
+        (xy 1.74117 -0.398145)
+        (xy 1.754505 -0.398145)
+        (xy 2.02692 0.352425)
+      ) (layer "B.SilkS") (width 0) (fill solid))
+  )
